File: MicroTracker/Tracker/Power.sch (KiCad schematic (older format))
At the start: 8 parts, among them J1 Screw_Terminal_01x02, SW1 SW_SPDT, U1 LD1117S33TR_SOT223

Commit message: assigned parts
Parts:
- J1: footprint (none) -> Sparkfun-Artemis:AMASS_XT60-M
- SW1: footprint (none) -> Sparkfun-Artemis:SW_MLL1200S
Changed lines of the file:
@@
 F 0 "J1" V 5464 1662 50  0000 R CNN
 F 1 "Screw_Terminal_01x02" V 5373 1662 50  0000 R CNN
-F 2 "" H 5500 1850 50  0001 C CNN
+F 2 "Sparkfun-Artemis:AMASS_XT60-M" H 5500 1850 50  0001 C CNN
 F 3 "~" H 5500 1850 50  0001 C CNN
 	1    5500 1850
@@
 F 0 "SW1" H 5800 2985 50  0000 C CNN
 F 1 "SW_SPDT" H 5800 2894 50  0000 C CNN
-F 2 "" H 5800 2700 50  0001 C CNN
+F 2 "Sparkfun-Artemis:SW_MLL1200S" H 5800 2700 50  0001 C CNN
 F 3 "~" H 5800 2700 50  0001 C CNN
 	1    5800 2700

Commit message: fixed errors
Connections:
- net at J1.2 (Pin_2), SW1.2 (B): no longer D1.1 (K)
- net at SW1.1 (A): now also D1.1 (K)
- no-connect marks 0 -> 1
Changed lines of the file:
@@
 L power:GND #PWR0101
 U 1 1 5EFA8BC9
-P 5500 2150
-F 0 "#PWR0101" H 5500 1900 50  0001 C CNN
-F 1 "GND" H 5505 1977 50  0000 C CNN
-F 2 "" H 5500 2150 50  0001 C CNN
-F 3 "" H 5500 2150 50  0001 C CNN
-	1    5500 2150
+P 5500 2250
+F 0 "#PWR0101" H 5500 2000 50  0001 C CNN
+F 1 "GND" H 5505 2077 50  0000 C CNN
+F 2 "" H 5500 2250 50  0001 C CNN
+F 3 "" H 5500 2250 50  0001 C CNN
+	1    5500 2250
 	1    0    0    -1
 $EndComp
@@
 	1    0    0    -1
 $EndComp
-Wire Wire Line
-	5500 2050 5500 2100
 Wire Wire Line
 	5600 2050 5600 2100
@@
 	6700 5400 6700 5100
 Wire Wire Line
-	5600 2700 5600 3200
-Connection ~ 5600 2700
-Wire Wire Line
 	6150 5400 6700 5400
 Connection ~ 6150 5400
@@
 	6700 4350 6700 3900
 Connection ~ 6700 4350
-$Comp
-L power:PWR_FLAG #FLG0101
-U 1 1 5EFC14FC
-P 5500 2100
-F 0 "#FLG0101" H 5500 2175 50  0001 C CNN
-F 1 "PWR_FLAG" V 5500 2227 50  0000 L CNN
-F 2 "" H 5500 2100 50  0001 C CNN
-F 3 "~" H 5500 2100 50  0001 C CNN
-	1    5500 2100
-	0    -1   -1   0
-$EndComp
-Connection ~ 5500 2100
-Wire Wire Line
-	5500 2100 5500 2150
 $Comp
 L power:PWR_FLAG #FLG0102
@@
 Wire Wire Line
 	5150 3900 4800 3900
+Wire Wire Line
+	5500 2050 5500 2100
+$Comp
+L power:PWR_FLAG #FLG0101
+U 1 1 5F0CCCAB
+P 5500 2100
+F 0 "#FLG0101" H 5500 2175 50  0001 C CNN
+F 1 "PWR_FLAG" H 5500 2273 50  0000 C CNN
+F 2 "" H 5500 2100 50  0001 C CNN
+F 3 "~" H 5500 2100 50  0001 C CNN
+	1    5500 2100
+	0    -1   -1   0
+$EndComp
+Connection ~ 5500 2100
+Wire Wire Line
+	5500 2100 5500 2250
+Wire Wire Line
+	5600 3200 5600 3100
+Wire Wire Line
+	5600 3100 6350 3100
+Wire Wire Line
+	6350 3100 6350 2600
+Wire Wire Line
+	6350 2600 6000 2600
+NoConn ~ 6000 2800
 $EndSCHEMATC
