File: MicroTracker/Tracker/USB.sch (KiCad schematic (older format))
At the start: 3 parts, among them J3 USB_A, U7 CP2104

Commit message: assigned parts
Parts:
- added U12: TPD2EUSB30, Package_TO_SOT_SMD:Texas_DRT-3, symbol Power_Protection:TPD2EUSB30
- J3: footprint (none) -> Connector_USB:USB_Micro-B_Amphenol_10103594-0001LF_Horizontal
Connections:
- net GND: now also U7.2 (GND), U7.25 (PAD), U12.3 (GND)
- net at J3.2 (D-), U7.3 (D+): now also U12.2 (D-)
- net at J3.3 (D+), U7.4 (D-): now also U12.1 (D+)
- no-connect marks 0 -> 14
Other:
- moved on the sheet: J3
Changed lines of the file:
@@
 L Connector:USB_A J3
 U 1 1 5EF962A4
-P 3550 3000
-F 0 "J3" H 3607 3467 50  0000 C CNN
-F 1 "USB_A" H 3607 3376 50  0000 C CNN
-F 2 "" H 3700 2950 50  0001 C CNN
-F 3 " ~" H 3700 2950 50  0001 C CNN
-	1    3550 3000
+P 2600 3000
+F 0 "J3" H 2657 3467 50  0000 C CNN
+F 1 "USB_A" H 2657 3376 50  0000 C CNN
+F 2 "Connector_USB:USB_Micro-B_Amphenol_10103594-0001LF_Horizontal" H 2750 2950 50  0001 C CNN
+F 3 " ~" H 2750 2950 50  0001 C CNN
+	1    2600 3000
 	1    0    0    -1
 $EndComp
@@
 L power:GND #PWR0121
 U 1 1 5EF97340
-P 3550 3550
-F 0 "#PWR0121" H 3550 3300 50  0001 C CNN
-F 1 "GND" H 3555 3377 50  0000 C CNN
-F 2 "" H 3550 3550 50  0001 C CNN
-F 3 "" H 3550 3550 50  0001 C CNN
-	1    3550 3550
+P 2600 3550
+F 0 "#PWR0121" H 2600 3300 50  0001 C CNN
+F 1 "GND" H 2605 3377 50  0000 C CNN
+F 2 "" H 2600 3550 50  0001 C CNN
+F 3 "" H 2600 3550 50  0001 C CNN
+	1    2600 3550
 	1    0    0    -1
 $EndComp
 Wire Wire Line
-	3550 3550 3550 3400
+	2600 3550 2600 3400
 $Comp
 L Interface_USB:CP2104 U7
@@
 	1    0    0    -1
 $EndComp
-Wire Wire Line
-	4850 3000 3850 3000
-Wire Wire Line
-	3850 3100 4850 3100
 Text HLabel 6500 2700 2    50   Input ~ 0
 USB_DTR
@@
 Wire Wire Line
 	5350 2150 4700 2150
+$Comp
+L Power_Protection:TPD2EUSB30 U12
+U 1 1 5F15C012
+P 3350 3500
+F 0 "U12" H 3350 3867 50  0000 C CNN
+F 1 "TPD2EUSB30" H 3350 3776 50  0000 C CNN
+F 2 "Package_TO_SOT_SMD:Texas_DRT-3" H 2600 3200 50  0001 C CNN
+F 3 "http://www.ti.com/lit/ds/symlink/tpd2eusb30a.pdf" H 3350 3500 50  0001 C CNN
+	1    3350 3500
+	1    0    0    -1
+$EndComp
+$Comp
+L power:GND #PWR0169
+U 1 1 5F163599
+P 3350 4000
+F 0 "#PWR0169" H 3350 3750 50  0001 C CNN
+F 1 "GND" H 3355 3827 50  0000 C CNN
+F 2 "" H 3350 4000 50  0001 C CNN
+F 3 "" H 3350 4000 50  0001 C CNN
+	1    3350 4000
+	1    0    0    -1
+$EndComp
+Wire Wire Line
+	3750 3500 3750 3100
+Wire Wire Line
+	2900 3100 3750 3100
+Connection ~ 3750 3100
+Wire Wire Line
+	3750 3100 4850 3100
+Wire Wire Line
+	2950 3500 2950 3000
+Wire Wire Line
+	2900 3000 2950 3000
+Connection ~ 2950 3000
+Wire Wire Line
+	2950 3000 4850 3000
+Wire Wire Line
+	3350 3900 3350 4000
+NoConn ~ 4850 2700
+NoConn ~ 2900 2800
+NoConn ~ 4850 3300
+NoConn ~ 4850 3400
+NoConn ~ 4850 3500
+NoConn ~ 4850 3600
+NoConn ~ 4850 3800
+NoConn ~ 6250 3800
+NoConn ~ 6250 3700
+NoConn ~ 6250 3600
+NoConn ~ 6250 3400
+NoConn ~ 6250 3300
+NoConn ~ 6250 2600
+NoConn ~ 6250 2500
+$Comp
+L power:GND #PWR0170
+U 1 1 5F167400
+P 5550 4400
+F 0 "#PWR0170" H 5550 4150 50  0001 C CNN
+F 1 "GND" H 5555 4227 50  0000 C CNN
+F 2 "" H 5550 4400 50  0001 C CNN
+F 3 "" H 5550 4400 50  0001 C CNN
+	1    5550 4400
+	1    0    0    -1
+$EndComp
+Wire Wire Line
+	5550 4100 5550 4300
+Wire Wire Line
+	5650 4100 5650 4300
+Wire Wire Line
+	5650 4300 5550 4300
+Connection ~ 5550 4300
+Wire Wire Line
+	5550 4300 5550 4400
 $EndSCHEMATC

Commit message: fixed errors
Connections:
- no-connect marks 14 -> 17
Changed lines of the file:
@@
 Wire Wire Line
 	5550 4300 5550 4400
+NoConn ~ 2500 3400
+NoConn ~ 6250 2800
+NoConn ~ 5750 2200
 $EndSCHEMATC
